File: LV/RPDM v2/5V_Converters.sch (KiCad schematic (older format))
At the start: 26 parts

Commit message: RPDM v2 nearly done
Parts:
- removed C? (x4): C, symbol Device:C
- removed C? (x4): CP, symbol Device:CP
- removed D? (x2): LED, symbol Device:LED
- removed F? (x2): Fuse, symbol Device:Fuse
- removed Q? (x4): Q_NPN_BCE, symbol Device:Q_NPN_BCE
- removed R? (x4): 22k, symbol Device:R
- removed R? (x2): 47k, symbol Device:R
- removed R? (x2): 1.8k, symbol Device:R
- removed U? (x2): OKI-78SR-5_1.5-W36-C, Converter_DCDC:Converter_DCDC_muRata_OKI-78SR_Vertical, symbol RPDM-v2-rescue:OKI-78SR-5_1.5-W36-C-Converter_DCDC-RPDM-v1-rescue
Other:
- note added: "5V DCDC Converters"
- note removed: "5V DCDC Converters\n\n"
- note removed: "LED Fuse Indicators\n"
