File: LV/RPDM v2/TSAL_Logic.sch (KiCad schematic (older format))
At the start: 13 parts

Commit message: rpdm
Parts:
- removed R?: 20k, symbol Device:RTRIM
- added RV?: 20kΩ, symbol Device2:R_Potentiometer_Trim
- gave numbers to parts that had none: 12
Connections:
- net at C2603.1, U2601.2 (TR), U2601.6 (THR): now also RV?.2
- net at R2608.2: now also RV?.3
Other:
- moved on the sheet: C2603, R2603
