File: LV/RPDM v2/Relay.sch (KiCad schematic (older format))
At the start: 4 parts

Commit message: rpdm
Parts:
- gave numbers to parts that had none: 4
Other:
- moved on the sheet: D2501, K2501, Q2501, R2501
Changed lines of the file:
@@
 $Descr A4 11693 8268
 encoding utf-8
-Sheet 24 30
+Sheet 25 30
 Title "Relay Circuit"
 Date "2021-06-28"
@@
 L Relay:G5LE-1 K?
 U 1 1 5E5EE7C7
-P 5700 2100
+P 5600 3150
 AR Path="/5E554D5D/5E5EE7C7" Ref="K?"  Part="1"
-AR Path="/5E554D5D/5E5E9CA9/5E5EE7C7" Ref="K?"  Part="1"
+AR Path="/5E554D5D/5E5E9CA9/5E5EE7C7" Ref="K2501"  Part="1"
 AR Path="/5E554D5D/5E5A0290/5E5EE7C7" Ref="K?"  Part="1"
 AR Path="/5E554D5D/5E5A035E/5E5EE7C7" Ref="K?"  Part="1"
@@
 AR Path="/5E554D5D/60DE7B67/5E5EE7C7" Ref="K?"  Part="1"
 AR Path="/5E554D5D/60DE7FBD/5E5EE7C7" Ref="K?"  Part="1"
-AR Path="/5E554D5D/60DE88EB/5E5EE7C7" Ref="K?"  Part="1"
-AR Path="/5E554D5D/60DED789/5E5EE7C7" Ref="K?"  Part="1"
-AR Path="/5E554D5D/60DEDCB5/5E5EE7C7" Ref="K?"  Part="1"
-F 0 "K?" V 5133 2100 50  0000 C CNN
-F 1 "G5LE-1" V 5224 2100 50  0000 C CNN
-F 2 "Relay_THT:Relay_SPDT_Omron-G5LE-1" H 6150 2050 50  0001 L CNN
-F 3 "http://www.omron.com/ecb/products/pdf/en-g5le.pdf" H 5700 2100 50  0001 C CNN
-	1    5700 2100
+AR Path="/5E554D5D/60DE88EB/5E5EE7C7" Ref="K2201"  Part="1"
+AR Path="/5E554D5D/60DED789/5E5EE7C7" Ref="K2301"  Part="1"
+AR Path="/5E554D5D/60DEDCB5/5E5EE7C7" Ref="K2401"  Part="1"
+AR Path="/60E5EBEF/5E5EE7C7" Ref="K?"  Part="1"
+F 0 "K2501" V 6050 3150 50  0000 C CNN
+F 1 "G5LE-1" V 5124 3150 50  0000 C CNN
+F 2 "Relay_THT:Relay_SPDT_Omron-G5LE-1" H 6050 3100 50  0001 L CNN
+F 3 "http://www.omron.com/ecb/products/pdf/en-g5le.pdf" H 5600 3150 50  0001 C CNN
+	1    5600 3150
 	0    1    -1   0
 $EndComp
@@
 L Device:D D?
 U 1 1 5E5EE7CD
-P 5550 2750
+P 5600 3800
 AR Path="/5E554D5D/5E5EE7CD" Ref="D?"  Part="1"
-AR Path="/5E554D5D/5E5E9CA9/5E5EE7CD" Ref="D?"  Part="1"
+AR Path="/5E554D5D/5E5E9CA9/5E5EE7CD" Ref="D2501"  Part="1"
 AR Path="/5E554D5D/5E5A0290/5E5EE7CD" Ref="D?"  Part="1"
 AR Path="/5E554D5D/5E5A035E/5E5EE7CD" Ref="D?"  Part="1"
@@
 AR Path="/5E554D5D/60DE7B67/5E5EE7CD" Ref="D?"  Part="1"
 AR Path="/5E554D5D/60DE7FBD/5E5EE7CD" Ref="D?"  Part="1"
-AR Path="/5E554D5D/60DE88EB/5E5EE7CD" Ref="D?"  Part="1"
-AR Path="/5E554D5D/60DED789/5E5EE7CD" Ref="D?"  Part="1"
-AR Path="/5E554D5D/60DEDCB5/5E5EE7CD" Ref="D?"  Part="1"
-F 0 "D?" H 5550 2950 50  0000 C CNN
-F 1 "D" H 5550 2850 50  0000 C CNN
-F 2 "" H 5550 2750 50  0001 C CNN
-F 3 "~" H 5550 2750 50  0001 C CNN
-	1    5550 2750
+AR Path="/5E554D5D/60DE88EB/5E5EE7CD" Ref="D2201"  Part="1"
+AR Path="/5E554D5D/60DED789/5E5EE7CD" Ref="D2301"  Part="1"
+AR Path="/5E554D5D/60DEDCB5/5E5EE7CD" Ref="D2401"  Part="1"
+AR Path="/60E5EBEF/5E5EE7CD" Ref="D?"  Part="1"
+F 0 "D2501" H 5600 4000 50  0000 C CNN
+F 1 "D" H 5600 3900 50  0000 C CNN
+F 2 "" H 5600 3800 50  0001 C CNN
+F 3 "~" H 5600 3800 50  0001 C CNN
+	1    5600 3800
 	1    0    0    1
 $EndComp
 Wire Wire Line
-	5700 2750 6100 2750
+	5750 3800 6000 3800
 Wire Wire Line
-	6100 2750 6100 2300
+	6000 3800 6000 3350
 Wire Wire Line
-	6100 2300 6000 2300
+	6000 3350 5900 3350
 Wire Wire Line
-	5400 2300 5300 2300
+	5300 3350 5200 3350
 Wire Wire Line
-	5300 2300 5300 2750
+	5200 3350 5200 3800
 Wire Wire Line
-	5300 2750 5400 2750
-Text HLabel 5100 1900 0    50   Input ~ 0
+	5200 3800 5450 3800
+Text HLabel 5000 2950 0    50   Input ~ 0
 Vin
-NoConn ~ 6000 2000
-Text HLabel 6350 1800 2    50   Input ~ 0
+NoConn ~ 5900 3050
+Text HLabel 6000 2850 2    50   Input ~ 0
 Output
 $Comp
-L Device:Q_NPN_BCE Q?
+L Device:Q_NPN_BCE Q2501
 U 1 1 5E5F1342
-P 6000 3050
-AR Path="/5E554D5D/5E5E9CA9/5E5F1342" Ref="Q?"  Part="1"
+P 5900 4200
+AR Path="/5E554D5D/5E5E9CA9/5E5F1342" Ref="Q2501"  Part="1"
 AR Path="/5E554D5D/5E5A0290/5E5F1342" Ref="Q?"  Part="1"
 AR Path="/5E554D5D/5E5A035E/5E5F1342" Ref="Q?"  Part="1"
@@
 AR Path="/5E554D5D/60DE7B67/5E5F1342" Ref="Q?"  Part="1"
 AR Path="/5E554D5D/60DE7FBD/5E5F1342" Ref="Q?"  Part="1"
-AR Path="/5E554D5D/60DE88EB/5E5F1342" Ref="Q?"  Part="1"
-AR Path="/5E554D5D/60DED789/5E5F1342" Ref="Q?"  Part="1"
-AR Path="/5E554D5D/60DEDCB5/5E5F1342" Ref="Q?"  Part="1"
-F 0 "Q?" H 6191 3096 50  0000 L CNN
-F 1 "Q_NPN_BCE" H 6191 3005 50  0000 L CNN
-F 2 "" H 6200 3150 50  0001 C CNN
-F 3 "~" H 6000 3050 50  0001 C CNN
-	1    6000 3050
+AR Path="/5E554D5D/60DE88EB/5E5F1342" Ref="Q2201"  Part="1"
+AR Path="/5E554D5D/60DED789/5E5F1342" Ref="Q2301"  Part="1"
+AR Path="/5E554D5D/60DEDCB5/5E5F1342" Ref="Q2401"  Part="1"
+AR Path="/60E5EBEF/5E5F1342" Ref="Q?"  Part="1"
+F 0 "Q2501" H 6091 4246 50  0000 L CNN
+F 1 "Q_NPN_BCE" H 6091 4155 50  0000 L CNN
+F 2 "" H 6100 4300 50  0001 C CNN
+F 3 "~" H 5900 4200 50  0001 C CNN
+	1    5900 4200
 	1    0    0    -1
 $EndComp
 $Comp
-L Device:R R?
+L Device:R R2501
 U 1 1 5E5F2921
-P 5550 3050
-AR Path="/5E554D5D/5E5E9CA9/5E5F2921" Ref="R?"  Part="1"
+P 5450 4200
+AR Path="/5E554D5D/5E5E9CA9/5E5F2921" Ref="R2501"  Part="1"
 AR Path="/5E554D5D/5E5A0290/5E5F2921" Ref="R?"  Part="1"
 AR Path="/5E554D5D/5E5A035E/5E5F2921" Ref="R?"  Part="1"
@@
 AR Path="/5E554D5D/60DE7B67/5E5F2921" Ref="R?"  Part="1"
 AR Path="/5E554D5D/60DE7FBD/5E5F2921" Ref="R?"  Part="1"
-AR Path="/5E554D5D/60DE88EB/5E5F2921" Ref="R?"  Part="1"
-AR Path="/5E554D5D/60DED789/5E5F2921" Ref="R?"  Part="1"
-AR Path="/5E554D5D/60DEDCB5/5E5F2921" Ref="R?"  Part="1"
-F 0 "R?" V 5350 3050 50  0000 C CNN
-F 1 "R" V 5450 3050 50  0000 C CNN
-F 2 "" V 5480 3050 50  0001 C CNN
-F 3 "~" H 5550 3050 50  0001 C CNN
-	1    5550 3050
+AR Path="/5E554D5D/60DE88EB/5E5F2921" Ref="R2201"  Part="1"
+AR Path="/5E554D5D/60DED789/5E5F2921" Ref="R2301"  Part="1"
+AR Path="/5E554D5D/60DEDCB5/5E5F2921" Ref="R2401"  Part="1"
+AR Path="/60E5EBEF/5E5F2921" Ref="R?"  Part="1"
+F 0 "R2501" V 5250 4200 50  0000 C CNN
+F 1 "R" V 5350 4200 50  0000 C CNN
+F 2 "" V 5380 4200 50  0001 C CNN
+F 3 "~" H 5450 4200 50  0001 C CNN
+	1    5450 4200
 	0    1    -1   0
 $EndComp
 Wire Wire Line
-	6000 1800 6350 1800
+	5900 2850 6000 2850
 $Comp
-L power:GND #PWR?
+L power:GND #PWR02501
 U 1 1 5E5F4802
-P 6100 3350
-AR Path="/5E554D5D/5E5E9CA9/5E5F4802" Ref="#PWR?"  Part="1"
+P 6000 4500
+AR Path="/5E554D5D/5E5E9CA9/5E5F4802" Ref="#PWR02501"  Part="1"
 AR Path="/5E554D5D/5E5A0290/5E5F4802" Ref="#PWR?"  Part="1"
 AR Path="/5E554D5D/5E5A035E/5E5F4802" Ref="#PWR?"  Part="1"
@@
 AR Path="/5E554D5D/60DE7B67/5E5F4802" Ref="#PWR?"  Part="1"
 AR Path="/5E554D5D/60DE7FBD/5E5F4802" Ref="#PWR?"  Part="1"
-AR Path="/5E554D5D/60DE88EB/5E5F4802" Ref="#PWR?"  Part="1"
-AR Path="/5E554D5D/60DED789/5E5F4802" Ref="#PWR?"  Part="1"
-AR Path="/5E554D5D/60DEDCB5/5E5F4802" Ref="#PWR?"  Part="1"
-F 0 "#PWR?" H 6100 3100 50  0001 C CNN
-F 1 "GND" H 6105 3177 50  0000 C CNN
-F 2 "" H 6100 3350 50  0001 C CNN
-F 3 "" H 6100 3350 50  0001 C CNN
-	1    6100 3350
+AR Path="/5E554D5D/60DE88EB/5E5F4802" Ref="#PWR02201"  Part="1"
+AR Path="/5E554D5D/60DED789/5E5F4802" Ref="#PWR02301"  Part="1"
+AR Path="/5E554D5D/60DEDCB5/5E5F4802" Ref="#PWR02401"  Part="1"
+AR Path="/60E5EBEF/5E5F4802" Ref="#PWR?"  Part="1"
+F 0 "#PWR02501" H 6000 4250 50  0001 C CNN
+F 1 "GND" H 6005 4327 50  0000 C CNN
+F 2 "" H 6000 4500 50  0001 C CNN
+F 3 "" H 6000 4500 50  0001 C CNN
+	1    6000 4500
 	-1   0    0    -1
 $EndComp
-Connection ~ 5300 2300
+Connection ~ 5200 3350
 Wire Wire Line
-	5100 1900 5300 1900
+	5000 2950 5200 2950
 Wire Wire Line
-	5300 1900 5300 2300
-Text HLabel 5100 3050 0    50   Input ~ 0
+	5200 2950 5200 3350
+Text HLabel 5000 4200 0    50   Input ~ 0
 Trigger
 Wire Wire Line
-	5400 1900 5300 1900
-Connection ~ 5300 1900
+	5300 2950 5200 2950
+Connection ~ 5200 2950
 Wire Wire Line
-	6100 3350 6100 3250
+	6000 4500 6000 4400
 Wire Wire Line
-	6100 2850 6100 2750
-Connection ~ 6100 2750
+	6000 4000 6000 3800
+Connection ~ 6000 3800
 Wire Wire Line
-	5800 3050 5700 3050
+	5700 4200 5600 4200
 Wire Wire Line
-	5400 3050 5100 3050
+	5300 4200 5000 4200
 $EndSCHEMATC

Commit message: rpdm
Parts:
- removed Q2501: Q_NPN_BCE, symbol Device:Q_NPN_BCE
- removed R2501: R, symbol Device:R
- added Q?: Q_Dual_NMOS_S1G1S2G2D2D2D1D1, symbol Device2:Q_Dual_NMOS_S1G1S2G2D2D2D1D1
- added R24: 100k, symbol Device2:R
- renumbered D2501 to D24, K2501 to K4
Connections:
- net GND: now also Q?.1 (S), R24.2
- net Trigger: now also Q?.2 (G), R24.1
- net at D24.2 (A), K4.5: now also Q?.7 (D), Q?.8 (D)
Other:
- moved on the sheet: D24, K4
Changed lines of the file:
@@
 $Descr A4 11693 8268
 encoding utf-8
-Sheet 25 29
+Sheet 28 32
 Title "Relay Circuit"
 Date "2021-06-28"
@@
 L Relay:G5LE-1 K?
 U 1 1 5E5EE7C7
-P 5600 3150
+P 5600 3300
 AR Path="/5E554D5D/5E5EE7C7" Ref="K?"  Part="1"
-AR Path="/5E554D5D/5E5E9CA9/5E5EE7C7" Ref="K2501"  Part="1"
+AR Path="/5E554D5D/5E5E9CA9/5E5EE7C7" Ref="K4"  Part="1"
 AR Path="/5E554D5D/5E5A0290/5E5EE7C7" Ref="K?"  Part="1"
 AR Path="/5E554D5D/5E5A035E/5E5EE7C7" Ref="K?"  Part="1"
@@
 AR Path="/5E554D5D/60DE7B67/5E5EE7C7" Ref="K?"  Part="1"
 AR Path="/5E554D5D/60DE7FBD/5E5EE7C7" Ref="K?"  Part="1"
-AR Path="/5E554D5D/60DE88EB/5E5EE7C7" Ref="K2201"  Part="1"
-AR Path="/5E554D5D/60DED789/5E5EE7C7" Ref="K2301"  Part="1"
-AR Path="/5E554D5D/60DEDCB5/5E5EE7C7" Ref="K2401"  Part="1"
+AR Path="/5E554D5D/60DE88EB/5E5EE7C7" Ref="K1"  Part="1"
+AR Path="/5E554D5D/60DED789/5E5EE7C7" Ref="K2"  Part="1"
+AR Path="/5E554D5D/60DEDCB5/5E5EE7C7" Ref="K3"  Part="1"
 AR Path="/60E5EBEF/5E5EE7C7" Ref="K?"  Part="1"
-F 0 "K2501" V 6050 3150 50  0000 C CNN
-F 1 "G5LE-1" V 5124 3150 50  0000 C CNN
-F 2 "Relay_THT:Relay_SPDT_Omron-G5LE-1" H 6050 3100 50  0001 L CNN
-F 3 "http://www.omron.com/ecb/products/pdf/en-g5le.pdf" H 5600 3150 50  0001 C CNN
-	1    5600 3150
+F 0 "K4" V 6050 3300 50  0000 C CNN
+F 1 "G5LE-1" V 5124 3300 50  0000 C CNN
+F 2 "Relay_THT:Relay_SPDT_Omron-G5LE-1" H 6050 3250 50  0001 L CNN
+F 3 "http://www.omron.com/ecb/products/pdf/en-g5le.pdf" H 5600 3300 50  0001 C CNN
+	1    5600 3300
 	0    1    -1   0
 $EndComp
@@
 L Device:D D?
 U 1 1 5E5EE7CD
-P 5600 3800
+P 5600 4000
 AR Path="/5E554D5D/5E5EE7CD" Ref="D?"  Part="1"
-AR Path="/5E554D5D/5E5E9CA9/5E5EE7CD" Ref="D2501"  Part="1"
+AR Path="/5E554D5D/5E5E9CA9/5E5EE7CD" Ref="D24"  Part="1"
 AR Path="/5E554D5D/5E5A0290/5E5EE7CD" Ref="D?"  Part="1"
 AR Path="/5E554D5D/5E5A035E/5E5EE7CD" Ref="D?"  Part="1"
@@
 AR Path="/5E554D5D/60DE7B67/5E5EE7CD" Ref="D?"  Part="1"
 AR Path="/5E554D5D/60DE7FBD/5E5EE7CD" Ref="D?"  Part="1"
-AR Path="/5E554D5D/60DE88EB/5E5EE7CD" Ref="D2201"  Part="1"
-AR Path="/5E554D5D/60DED789/5E5EE7CD" Ref="D2301"  Part="1"
-AR Path="/5E554D5D/60DEDCB5/5E5EE7CD" Ref="D2401"  Part="1"
+AR Path="/5E554D5D/60DE88EB/5E5EE7CD" Ref="D21"  Part="1"
+AR Path="/5E554D5D/60DED789/5E5EE7CD" Ref="D22"  Part="1"
+AR Path="/5E554D5D/60DEDCB5/5E5EE7CD" Ref="D23"  Part="1"
 AR Path="/60E5EBEF/5E5EE7CD" Ref="D?"  Part="1"
-F 0 "D2501" H 5600 4000 50  0000 C CNN
-F 1 "D" H 5600 3900 50  0000 C CNN
-F 2 "" H 5600 3800 50  0001 C CNN
-F 3 "~" H 5600 3800 50  0001 C CNN
-	1    5600 3800
+F 0 "D24" H 5600 4200 50  0000 C CNN
+F 1 "D" H 5600 4100 50  0000 C CNN
+F 2 "" H 5600 4000 50  0001 C CNN
+F 3 "~" H 5600 4000 50  0001 C CNN
+	1    5600 4000
 	1    0    0    1
 $EndComp
 Wire Wire Line
-	5750 3800 6000 3800
+	5750 4000 6000 4000
 Wire Wire Line
-	6000 3800 6000 3350
+	6000 4000 6000 3500
 Wire Wire Line
-	6000 3350 5900 3350
+	6000 3500 5900 3500
 Wire Wire Line
-	5300 3350 5200 3350
+	5300 3500 5200 3500
 Wire Wire Line
-	5200 3350 5200 3800
+	5200 3500 5200 4000
 Wire Wire Line
-	5200 3800 5450 3800
-Text HLabel 5000 2950 0    50   Input ~ 0
+	5200 4000 5450 4000
+Text HLabel 5000 3100 0    50   Input ~ 0
 Vin
-NoConn ~ 5900 3050
-Text HLabel 6000 2850 2    50   Input ~ 0
+NoConn ~ 5900 3200
+Text HLabel 6000 3000 2    50   Input ~ 0
 Output
+Wire Wire Line
+	5900 3000 6000 3000
 $Comp
-L Device:Q_NPN_BCE Q2501
-U 1 1 5E5F1342
-P 5900 4200
-AR Path="/5E554D5D/5E5E9CA9/5E5F1342" Ref="Q2501"  Part="1"
-AR Path="/5E554D5D/5E5A0290/5E5F1342" Ref="Q?"  Part="1"
-AR Path="/5E554D5D/5E5A035E/5E5F1342" Ref="Q?"  Part="1"
-AR Path="/5E554D5D/5E5A09AA/5E5F1342" Ref="Q?"  Part="1"
-AR Path="/5E554D5D/5E5A0BF4/5E5F1342" Ref="Q?"  Part="1"
-AR Path="/5E554D5D/610FDB0E/5E5F1342" Ref="Q?"  Part="1"
-AR Path="/5E554D5D/60DE75D7/5E5F1342" Ref="Q?"  Part="1"
-AR Path="/5E554D5D/60DE7B67/5E5F1342" Ref="Q?"  Part="1"
-AR Path="/5E554D5D/60DE7FBD/5E5F1342" Ref="Q?"  Part="1"
-AR Path="/5E554D5D/60DE88EB/5E5F1342" Ref="Q2201"  Part="1"
-AR Path="/5E554D5D/60DED789/5E5F1342" Ref="Q2301"  Part="1"
-AR Path="/5E554D5D/60DEDCB5/5E5F1342" Ref="Q2401"  Part="1"
-AR Path="/60E5EBEF/5E5F1342" Ref="Q?"  Part="1"
-F 0 "Q2501" H 6091 4246 50  0000 L CNN
-F 1 "Q_NPN_BCE" H 6091 4155 50  0000 L CNN
-F 2 "" H 6100 4300 50  0001 C CNN
-F 3 "~" H 5900 4200 50  0001 C CNN
-	1    5900 4200
-	1    0    0    -1
-$EndComp
-$Comp
-L Device:R R2501
-U 1 1 5E5F2921
-P 5450 4200
-AR Path="/5E554D5D/5E5E9CA9/5E5F2921" Ref="R2501"  Part="1"
-AR Path="/5E554D5D/5E5A0290/5E5F2921" Ref="R?"  Part="1"
-AR Path="/5E554D5D/5E5A035E/5E5F2921" Ref="R?"  Part="1"
-AR Path="/5E554D5D/5E5A09AA/5E5F2921" Ref="R?"  Part="1"
-AR Path="/5E554D5D/5E5A0BF4/5E5F2921" Ref="R?"  Part="1"
-AR Path="/5E554D5D/610FDB0E/5E5F2921" Ref="R?"  Part="1"
-AR Path="/5E554D5D/60DE75D7/5E5F2921" Ref="R?"  Part="1"
-AR Path="/5E554D5D/60DE7B67/5E5F2921" Ref="R?"  Part="1"
-AR Path="/5E554D5D/60DE7FBD/5E5F2921" Ref="R?"  Part="1"
-AR Path="/5E554D5D/60DE88EB/5E5F2921" Ref="R2201"  Part="1"
-AR Path="/5E554D5D/60DED789/5E5F2921" Ref="R2301"  Part="1"
-AR Path="/5E554D5D/60DEDCB5/5E5F2921" Ref="R2401"  Part="1"
-AR Path="/60E5EBEF/5E5F2921" Ref="R?"  Part="1"
-F 0 "R2501" V 5250 4200 50  0000 C CNN
-F 1 "R" V 5350 4200 50  0000 C CNN
-F 2 "" V 5380 4200 50  0001 C CNN
-F 3 "~" H 5450 4200 50  0001 C CNN
-	1    5450 4200
-	0    1    -1   0
-$EndComp
-Wire Wire Line
-	5900 2850 6000 2850
-$Comp
-L power:GND #PWR02501
+L power:GND #PWR032
 U 1 1 5E5F4802
-P 6000 4500
-AR Path="/5E554D5D/5E5E9CA9/5E5F4802" Ref="#PWR02501"  Part="1"
+P 6000 5000
+AR Path="/5E554D5D/5E5E9CA9/5E5F4802" Ref="#PWR032"  Part="1"
 AR Path="/5E554D5D/5E5A0290/5E5F4802" Ref="#PWR?"  Part="1"
 AR Path="/5E554D5D/5E5A035E/5E5F4802" Ref="#PWR?"  Part="1"
@@
 AR Path="/5E554D5D/60DE7B67/5E5F4802" Ref="#PWR?"  Part="1"
 AR Path="/5E554D5D/60DE7FBD/5E5F4802" Ref="#PWR?"  Part="1"
-AR Path="/5E554D5D/60DE88EB/5E5F4802" Ref="#PWR02201"  Part="1"
-AR Path="/5E554D5D/60DED789/5E5F4802" Ref="#PWR02301"  Part="1"
-AR Path="/5E554D5D/60DEDCB5/5E5F4802" Ref="#PWR02401"  Part="1"
+AR Path="/5E554D5D/60DE88EB/5E5F4802" Ref="#PWR026"  Part="1"
+AR Path="/5E554D5D/60DED789/5E5F4802" Ref="#PWR028"  Part="1"
+AR Path="/5E554D5D/60DEDCB5/5E5F4802" Ref="#PWR030"  Part="1"
 AR Path="/60E5EBEF/5E5F4802" Ref="#PWR?"  Part="1"
-F 0 "#PWR02501" H 6000 4250 50  0001 C CNN
-F 1 "GND" H 6005 4327 50  0000 C CNN
-F 2 "" H 6000 4500 50  0001 C CNN
-F 3 "" H 6000 4500 50  0001 C CNN
-	1    6000 4500
+F 0 "#PWR032" H 6000 4750 50  0001 C CNN
+F 1 "GND" H 6005 4827 50  0000 C CNN
+F 2 "" H 6000 5000 50  0001 C CNN
+F 3 "" H 6000 5000 50  0001 C CNN
+	1    6000 5000
 	-1   0    0    -1
 $EndComp
-Connection ~ 5200 3350
+Connection ~ 5200 3500
 Wire Wire Line
-	5000 2950 5200 2950
+	5000 3100 5200 3100
 Wire Wire Line
-	5200 2950 5200 3350
-Text HLabel 5000 4200 0    50   Input ~ 0
+	5200 3100 5200 3500
+Text HLabel 5000 4500 0    50   Input ~ 0
 Trigger
 Wire Wire Line
-	5300 2950 5200 2950
-Connection ~ 5200 2950
+	5300 3100 5200 3100
+Connection ~ 5200 3100
 Wire Wire Line
-	6000 4500 6000 4400
+	6000 5000 6000 4700
 Wire Wire Line
-	6000 4000 6000 3800
-Connection ~ 6000 3800
+	6000 4300 6000 4200
+Connection ~ 6000 4000
 Wire Wire Line
-	5700 4200 5600 4200
+	5000 4500 5600 4500
+$Comp
+L Device2:R R24
+U 1 1 6183CC28
+P 5600 4750
+AR Path="/5E554D5D/5E5E9CA9/6183CC28" Ref="R24"  Part="1"
+AR Path="/5E554D5D/60DED789/6183CC28" Ref="R22"  Part="1"
+AR Path="/5E554D5D/60DE88EB/6183CC28" Ref="R21"  Part="1"
+AR Path="/5E554D5D/60DEDCB5/6183CC28" Ref="R23"  Part="1"
+F 0 "R24" H 5670 4796 50  0000 L CNN
+F 1 "100k" H 5670 4705 50  0000 L CNN
+F 2 "" V 5530 4750 50  0001 C CNN
+F 3 "~" H 5600 4750 50  0001 C CNN
+	1    5600 4750
+	1    0    0    -1
+$EndComp
 Wire Wire Line
-	5300 4200 5000 4200
+	5600 4900 5600 5000
+$Comp
+L power:GND #PWR031
+U 1 1 6183F1F1
+P 5600 5000
+AR Path="/5E554D5D/5E5E9CA9/6183F1F1" Ref="#PWR031"  Part="1"
+AR Path="/5E554D5D/5E5A0290/6183F1F1" Ref="#PWR?"  Part="1"
+AR Path="/5E554D5D/5E5A035E/6183F1F1" Ref="#PWR?"  Part="1"
+AR Path="/5E554D5D/5E5A09AA/6183F1F1" Ref="#PWR?"  Part="1"
+AR Path="/5E554D5D/5E5A0BF4/6183F1F1" Ref="#PWR?"  Part="1"
+AR Path="/5E554D5D/610FDB0E/6183F1F1" Ref="#PWR?"  Part="1"
+AR Path="/5E554D5D/60DE75D7/6183F1F1" Ref="#PWR?"  Part="1"
+AR Path="/5E554D5D/60DE7B67/6183F1F1" Ref="#PWR?"  Part="1"
+AR Path="/5E554D5D/60DE7FBD/6183F1F1" Ref="#PWR?"  Part="1"
+AR Path="/5E554D5D/60DE88EB/6183F1F1" Ref="#PWR025"  Part="1"
+AR Path="/5E554D5D/60DED789/6183F1F1" Ref="#PWR027"  Part="1"
+AR Path="/5E554D5D/60DEDCB5/6183F1F1" Ref="#PWR029"  Part="1"
+AR Path="/60E5EBEF/6183F1F1" Ref="#PWR?"  Part="1"
+F 0 "#PWR031" H 5600 4750 50  0001 C CNN
+F 1 "GND" H 5605 4827 50  0000 C CNN
+F 2 "" H 5600 5000 50  0001 C CNN
+F 3 "" H 5600 5000 50  0001 C CNN
+	1    5600 5000
+	-1   0    0    -1
+$EndComp
+Wire Wire Line
+	5600 4600 5600 4500
+Connection ~ 5600 4500
+Wire Wire Line
+	5600 4500 5700 4500
+$Comp
+L Device2:Q_Dual_NMOS_S1G1S2G2D2D2D1D1 Q?
+U 1 1 61147348
+P 5900 4500
+F 0 "Q?" H 6188 4546 50  0000 L CNN
+F 1 "Q_Dual_NMOS_S1G1S2G2D2D2D1D1" H 6188 4455 50  0000 L CNN
+F 2 "" H 6100 4500 50  0001 C CNN
+F 3 "~" H 6100 4500 50  0001 C CNN
+	1    5900 4500
+	1    0    0    -1
+$EndComp
+Wire Wire Line
+	6100 4300 6100 4200
+Wire Wire Line
+	6100 4200 6000 4200
+Connection ~ 6000 4200
+Wire Wire Line
+	6000 4200 6000 4000
 $EndSCHEMATC
