File: LV/RPDM v2/12V_DCDC.sch (KiCad schematic (older format))
At the start: 10 parts, among them U201 i7A24045A033V-001-R

Commit message: rpdm
Parts:
- removed R202: 249Ω, symbol Device:R
- C2903: renamed from C203; value 22uF -> 22µF
- R2901: renamed from R201; value 50kΩ -> 20kΩ
- renumbered C201 to C2901, C202 to C2902, C204 to C2904, D201 to D2901, R203 to R2903, TP201 to TP2901, U201 to U2901
Connections:
- net labels added: 12V_OUT, 24V_IN
- net labels removed: Vin, Vout
- wire segments 46 -> 43
Other:
- moved on the sheet: C2903, C2904, D2901, R2903, TP2901
Changed lines of the file:
@@
 $Descr A4 11693 8268
 encoding utf-8
-Sheet 2 28
+Sheet 29 30
 Title "DC/DC Converter Circuit"
 Date "2021-06-28"
@@
 	5000 3800 5000 3950
 Connection ~ 5000 4100
-Text Notes 6450 3100 0    50   ~ 0
+Text Notes 6300 3100 0    50   ~ 0
 DCDC Output Voltage\nTest Point
 Text Notes 5250 4400 0    50   ~ 0
@@
 L Connector:TestPoint TP?
 U 1 1 5E7E7EDC
-P 6500 3300
+P 6350 3300
 AR Path="/5E546572/5E7E7EDC" Ref="TP?"  Part="1"
-AR Path="/5E545B2D/5E7E7EDC" Ref="TP201"  Part="1"
+AR Path="/5E545B2D/5E7E7EDC" Ref="TP2901"  Part="1"
 AR Path="/5E5461C2/5E7E7EDC" Ref="TP?"  Part="1"
-F 0 "TP201" H 6558 3418 50  0000 L CNN
-F 1 "TestPoint" H 6558 3327 50  0000 L CNN
-F 2 "" H 6700 3300 50  0001 C CNN
-F 3 "~" H 6700 3300 50  0001 C CNN
-	1    6500 3300
-	1    0    0    -1
-$EndComp
-Wire Wire Line
-	6500 3300 6500 3500
-Wire Wire Line
-	6200 3500 6500 3500
+F 0 "TP2901" H 6408 3418 50  0000 L CNN
+F 1 "TestPoint" H 6408 3327 50  0000 L CNN
+F 2 "" H 6550 3300 50  0001 C CNN
+F 3 "~" H 6550 3300 50  0001 C CNN
+	1    6350 3300
+	1    0    0    -1
+$EndComp
+Wire Wire Line
+	6350 3300 6350 3500
 Wire Wire Line
 	4400 3500 4400 3650
@@
 P 4400 3800
 AR Path="/5E546572/5E7A7C2F" Ref="C?"  Part="1"
-AR Path="/5E545B2D/5E7A7C2F" Ref="C201"  Part="1"
+AR Path="/5E545B2D/5E7A7C2F" Ref="C2901"  Part="1"
 AR Path="/5E5461C2/5E7A7C2F" Ref="C?"  Part="1"
-F 0 "C201" H 4400 4000 50  0000 L CNN
+F 0 "C2901" H 4400 4000 50  0000 L CNN
 F 1 "330µF" H 4400 3900 50  0000 L CNN
 F 2 "" H 4438 3650 50  0001 C CNN
@@
 P 4750 3800
 AR Path="/5E546572/5E7A88E4" Ref="C?"  Part="1"
-AR Path="/5E545B2D/5E7A88E4" Ref="C202"  Part="1"
+AR Path="/5E545B2D/5E7A88E4" Ref="C2902"  Part="1"
 AR Path="/5E5461C2/5E7A88E4" Ref="C?"  Part="1"
-F 0 "C202" H 4750 4000 50  0000 L CNN
+F 0 "C2902" H 4750 4000 50  0000 L CNN
 F 1 "22µF" H 4750 3900 50  0000 L CNN
 F 2 "" H 4788 3650 50  0001 C CNN
@@
 	4750 3500 4750 3650
 Text HLabel 4200 3500 0    70   Input ~ 14
-Vin
-$Comp
-L DCDC_TDK:i7A24045A033V U201
+24V_IN
+$Comp
+L DCDC_TDK:i7A24045A033V U2901
 U 1 1 60E5B9E9
 P 5600 3800
-F 0 "U201" H 5600 4365 50  0000 C CNN
+F 0 "U2901" H 5600 4365 50  0000 C CNN
 F 1 "i7A24045A033V-001-R" H 5600 4274 50  0000 C CNN
 F 2 "" H 5450 4100 50  0001 C CNN
@@
 Connection ~ 5000 3950
 Wire Wire Line
-	7300 3650 7300 3500
-Wire Wire Line
-	7950 4000 7950 4100
+	6800 3650 6800 3500
+Wire Wire Line
+	7450 4000 7450 4100
 $Comp
 L power:GND #PWR?
 U 1 1 610D36B1
-P 7950 4200
+P 7450 4200
 AR Path="/5E546572/610D36B1" Ref="#PWR?"  Part="1"
-AR Path="/5E545B2D/610D36B1" Ref="#PWR0202"  Part="1"
+AR Path="/5E545B2D/610D36B1" Ref="#PWR02902"  Part="1"
 AR Path="/5E5461C2/610D36B1" Ref="#PWR?"  Part="1"
-F 0 "#PWR0202" H 7950 3950 50  0001 C CNN
-F 1 "GND" H 7955 4027 50  0000 C CNN
-F 2 "" H 7950 4200 50  0001 C CNN
-F 3 "" H 7950 4200 50  0001 C CNN
-	1    7950 4200
+F 0 "#PWR02902" H 7450 3950 50  0001 C CNN
+F 1 "GND" H 7455 4027 50  0000 C CNN
+F 2 "" H 7450 4200 50  0001 C CNN
+F 3 "" H 7450 4200 50  0001 C CNN
+	1    7450 4200
 	1    0    0    -1
 $EndComp
@@
 L Device:LED D?
 U 1 1 5E7B7CF5
-P 7950 3850
+P 7450 3850
 AR Path="/5E546572/5E7B7CF5" Ref="D?"  Part="1"
-AR Path="/5E545B2D/5E7B7CF5" Ref="D201"  Part="1"
+AR Path="/5E545B2D/5E7B7CF5" Ref="D2901"  Part="1"
 AR Path="/5E5461C2/5E7B7CF5" Ref="D?"  Part="1"
-F 0 "D201" V 8050 3750 50  0000 C CNN
-F 1 "PWR_ON_LED" V 7950 3550 50  0000 C CNN
-F 2 "" H 7950 3850 50  0001 C CNN
-F 3 "~" H 7950 3850 50  0001 C CNN
-	1    7950 3850
+F 0 "D2901" V 7550 3700 50  0000 C CNN
+F 1 "PWR_ON_LED" V 7450 3550 50  0000 C CNN
+F 2 "" H 7450 3850 50  0001 C CNN
+F 3 "~" H 7450 3850 50  0001 C CNN
+	1    7450 3850
 	0    -1   -1   0
 $EndComp
-Text HLabel 7950 3500 2    70   Output ~ 14
-Vout
-Wire Wire Line
-	6500 3500 7000 3500
-Wire Wire Line
-	7000 3650 7000 3500
-Wire Wire Line
-	7300 3950 7300 4100
+Text HLabel 7450 3500 2    70   Output ~ 14
+12V_OUT
+Wire Wire Line
+	6500 3650 6500 3500
+Wire Wire Line
+	6800 3950 6800 4100
 Connection ~ 4750 3500
 Wire Wire Line
@@
 Wire Wire Line
 	4200 3500 4400 3500
-Connection ~ 6500 3500
-Wire Wire Line
-	7000 4100 7000 3950
+Wire Wire Line
+	6500 4100 6500 3950
 $Comp
 L Device:CP C?
 U 1 1 610E5B6D
-P 7300 3800
+P 6800 3800
 AR Path="/5E546572/610E5B6D" Ref="C?"  Part="1"
-AR Path="/5E545B2D/610E5B6D" Ref="C204"  Part="1"
+AR Path="/5E545B2D/610E5B6D" Ref="C2904"  Part="1"
 AR Path="/5E5461C2/610E5B6D" Ref="C?"  Part="1"
-F 0 "C204" H 7300 4000 50  0000 L CNN
-F 1 "330uF" H 7300 3900 50  0000 L CNN
-F 2 "" H 7338 3650 50  0001 C CNN
-F 3 "~" H 7300 3800 50  0001 C CNN
-	1    7300 3800
+F 0 "C2904" H 6800 4000 50  0000 L CNN
+F 1 "330uF" H 6800 3900 50  0000 L CNN
+F 2 "" H 6838 3650 50  0001 C CNN
+F 3 "~" H 6800 3800 50  0001 C CNN
+	1    6800 3800
 	1    0    0    -1
 $EndComp
@@
 L Device:C C?
 U 1 1 5E7CBE12
-P 7000 3800
+P 6500 3800
 AR Path="/5E546572/5E7CBE12" Ref="C?"  Part="1"
-AR Path="/5E545B2D/5E7CBE12" Ref="C203"  Part="1"
+AR Path="/5E545B2D/5E7CBE12" Ref="C2903"  Part="1"
 AR Path="/5E5461C2/5E7CBE12" Ref="C?"  Part="1"
-F 0 "C203" H 7000 4000 50  0000 L CNN
-F 1 "22uF" H 7000 3900 50  0000 L CNN
-F 2 "" H 7038 3650 50  0001 C CNN
-F 3 "~" H 7000 3800 50  0001 C CNN
-	1    7000 3800
-	1    0    0    -1
-$EndComp
-Wire Wire Line
-	6150 3800 6100 3800
-Wire Wire Line
-	6500 3800 6450 3800
-Wire Wire Line
-	6800 3800 6850 3800
-Wire Wire Line
-	6850 4100 7000 4100
-Connection ~ 6850 4100
-Wire Wire Line
-	6850 3800 6850 4100
-$Comp
-L Device2:R_Trim R201
+F 0 "C2903" H 6500 4000 50  0000 L CNN
+F 1 "22µF" H 6500 3900 50  0000 L CNN
+F 2 "" H 6538 3650 50  0001 C CNN
+F 3 "~" H 6500 3800 50  0001 C CNN
+	1    6500 3800
+	1    0    0    -1
+$EndComp
+Wire Wire Line
+	6200 3800 6100 3800
+$Comp
+L Device2:R_Trim R2901
 U 1 1 60DDD93E
-P 6300 3800
-F 0 "R201" V 6375 3750 50  0000 C CNN
-F 1 "50kΩ" V 6200 3850 50  0000 C CNN
-F 2 "" V 6230 3800 50  0001 C CNN
-F 3 "~" H 6300 3800 50  0001 C CNN
-	1    6300 3800
-	0    1    -1   0
-$EndComp
-$Comp
-L Device:R R?
-U 1 1 5E7B412C
-P 6650 3800
-AR Path="/5E546572/5E7B412C" Ref="R?"  Part="1"
-AR Path="/5E545B2D/5E7B412C" Ref="R202"  Part="1"
-AR Path="/5E5461C2/5E7B412C" Ref="R?"  Part="1"
-F 0 "R202" V 6725 3800 50  0000 C CNN
-F 1 "249Ω" V 6550 3800 50  0000 C CNN
-F 2 "" V 6580 3800 50  0001 C CNN
-F 3 "~" H 6650 3800 50  0001 C CNN
-	1    6650 3800
-	0    -1   -1   0
+P 6200 3950
+F 0 "R2901" H 6250 3975 50  0000 L TNN
+F 1 "20kΩ" H 6250 3900 50  0000 L TNN
+F 2 "" V 6130 3950 50  0001 C CNN
+F 3 "~" H 6200 3950 50  0001 C CNN
+	1    6200 3950
+	1    0    0    -1
 $EndComp
 $Comp
@@
 P 4200 4200
 AR Path="/5E546572/5E7AC91D" Ref="#PWR?"  Part="1"
-AR Path="/5E545B2D/5E7AC91D" Ref="#PWR0201"  Part="1"
+AR Path="/5E545B2D/5E7AC91D" Ref="#PWR02901"  Part="1"
 AR Path="/5E5461C2/5E7AC91D" Ref="#PWR?"  Part="1"
-F 0 "#PWR0201" H 4200 3950 50  0001 C CNN
+F 0 "#PWR02901" H 4200 3950 50  0001 C CNN
 F 1 "GND" H 4205 4027 50  0000 C CNN
 F 2 "" H 4200 4200 50  0001 C CNN
@@
 Wire Wire Line
 	4200 4100 4200 4200
-Connection ~ 7000 3500
-Connection ~ 7000 4100
-Connection ~ 7300 3500
-Wire Wire Line
-	7300 4100 7000 4100
-Wire Wire Line
-	7000 3500 7300 3500
-Wire Wire Line
-	7950 3650 7950 3700
-Wire Wire Line
-	7300 4100 7950 4100
-Connection ~ 7300 4100
-Connection ~ 7950 4100
-Wire Wire Line
-	7950 3650 7900 3650
+Connection ~ 6500 3500
+Connection ~ 6500 4100
+Connection ~ 6800 3500
+Wire Wire Line
+	6800 4100 6500 4100
+Wire Wire Line
+	6500 3500 6800 3500
+Wire Wire Line
+	7450 3650 7450 3700
+Wire Wire Line
+	6800 4100 7450 4100
+Connection ~ 6800 4100
+Connection ~ 7450 4100
+Wire Wire Line
+	7450 3650 7400 3650
 $Comp
 L Device:R R?
 U 1 1 60E34B0B
-P 7750 3650
+P 7250 3650
 AR Path="/5E546572/60E34B0B" Ref="R?"  Part="1"
-AR Path="/5E545B2D/60E34B0B" Ref="R203"  Part="1"
+AR Path="/5E545B2D/60E34B0B" Ref="R2903"  Part="1"
 AR Path="/5E5461C2/60E34B0B" Ref="R?"  Part="1"
-F 0 "R203" V 7825 3650 50  0000 C CNN
-F 1 "1.8kΩ" V 7650 3650 50  0000 C CNN
-F 2 "" V 7680 3650 50  0001 C CNN
-F 3 "~" H 7750 3650 50  0001 C CNN
-	1    7750 3650
+F 0 "R2903" V 7325 3650 50  0000 C CNN
+F 1 "1.8kΩ" V 7150 3650 50  0000 C CNN
+F 2 "" V 7180 3650 50  0001 C CNN
+F 3 "~" H 7250 3650 50  0001 C CNN
+	1    7250 3650
 	0    -1   -1   0
 $EndComp
 Wire Wire Line
-	7300 3500 7550 3500
-Wire Wire Line
-	7600 3650 7550 3650
-Wire Wire Line
-	7550 3650 7550 3500
-Connection ~ 7550 3500
-Wire Wire Line
-	7550 3500 7950 3500
-Wire Wire Line
-	6100 4100 6850 4100
-Wire Wire Line
-	7950 4100 7950 4200
+	6800 3500 7050 3500
+Wire Wire Line
+	7100 3650 7050 3650
+Wire Wire Line
+	7050 3650 7050 3500
+Connection ~ 7050 3500
+Wire Wire Line
+	7050 3500 7450 3500
+Wire Wire Line
+	6100 4100 6200 4100
+Wire Wire Line
+	7450 4100 7450 4200
+Connection ~ 6200 4100
+Wire Wire Line
+	6200 4100 6500 4100
+Connection ~ 6350 3500
+Wire Wire Line
+	6350 3500 6500 3500
+Wire Wire Line
+	6200 3500 6350 3500
 $EndSCHEMATC

Commit message: rpdm
Parts:
- C3: renamed from C2901; footprint (none) -> Capacitor_THT:CP_Radial_D10.0mm_P5.00mm
- C4: renamed from C2902; footprint (none) -> Capacitor_extra:C_Murata_KCM55
- C5: renamed from C2903; footprint (none) -> Capacitor_extra:C_Murata_KCM55
- C6: renamed from C2904; footprint (none) -> Capacitor_THT:CP_Radial_D10.0mm_P5.00mm
- R27: renamed from R2903; value 1.8kΩ -> 10k
- RV1: renamed from R2901; value 20kΩ -> 50k; symbol Device2:R_Trim -> Device2:R_Potentiometer_Trim
- TP4: renamed from TP2901; footprint (none) -> TestPoint:TestPoint_THTPad_1.0x1.0mm_Drill0.5mm
- U2: renamed from U2901; footprint (none) -> DCDC:i7A24045A033V
- renumbered D2901 to D29
Connections:
- wire segments 43 -> 44
- no-connect marks 0 -> 1
Other:
- moved on the sheet: C5, C6, D29, R27
Changed lines of the file:
@@
 $Descr A4 11693 8268
 encoding utf-8
-Sheet 29 29
+Sheet 30 32
 Title "DC/DC Converter Circuit"
 Date "2021-06-28"
@@
 P 6350 3300
 AR Path="/5E546572/5E7E7EDC" Ref="TP?"  Part="1"
-AR Path="/5E545B2D/5E7E7EDC" Ref="TP2901"  Part="1"
+AR Path="/5E545B2D/5E7E7EDC" Ref="TP4"  Part="1"
 AR Path="/5E5461C2/5E7E7EDC" Ref="TP?"  Part="1"
-F 0 "TP2901" H 6408 3418 50  0000 L CNN
+F 0 "TP4" H 6408 3418 50  0000 L CNN
 F 1 "TestPoint" H 6408 3327 50  0000 L CNN
-F 2 "" H 6550 3300 50  0001 C CNN
+F 2 "TestPoint:TestPoint_THTPad_1.0x1.0mm_Drill0.5mm" H 6550 3300 50  0001 C CNN
 F 3 "~" H 6550 3300 50  0001 C CNN
 	1    6350 3300
@@
 P 4400 3800
 AR Path="/5E546572/5E7A7C2F" Ref="C?"  Part="1"
-AR Path="/5E545B2D/5E7A7C2F" Ref="C2901"  Part="1"
+AR Path="/5E545B2D/5E7A7C2F" Ref="C3"  Part="1"
 AR Path="/5E5461C2/5E7A7C2F" Ref="C?"  Part="1"
-F 0 "C2901" H 4400 4000 50  0000 L CNN
+F 0 "C3" H 4400 4000 50  0000 L CNN
 F 1 "330µF" H 4400 3900 50  0000 L CNN
-F 2 "" H 4438 3650 50  0001 C CNN
-F 3 "~" H 4400 3800 50  0001 C CNN
+F 2 "Capacitor_THT:CP_Radial_D10.0mm_P5.00mm" H 4438 3650 50  0001 C CNN
+F 3 "https://content.kemet.com/datasheets/KEM_A4067_A750.pdf" H 4400 3800 50  0001 C CNN
 	1    4400 3800
 	1    0    0    -1
@@
 P 4750 3800
 AR Path="/5E546572/5E7A88E4" Ref="C?"  Part="1"
-AR Path="/5E545B2D/5E7A88E4" Ref="C2902"  Part="1"
+AR Path="/5E545B2D/5E7A88E4" Ref="C4"  Part="1"
 AR Path="/5E5461C2/5E7A88E4" Ref="C?"  Part="1"
-F 0 "C2902" H 4750 4000 50  0000 L CNN
+F 0 "C4" H 4750 4000 50  0000 L CNN
 F 1 "22µF" H 4750 3900 50  0000 L CNN
-F 2 "" H 4788 3650 50  0001 C CNN
-F 3 "~" H 4750 3800 50  0001 C CNN
+F 2 "Capacitor_extra:C_Murata_KCM55" H 4788 3650 50  0001 C CNN
+F 3 "https://search.murata.co.jp/Ceramy/image/img/A01X/G101/ENG/KCM55_E.pdf" H 4750 3800 50  0001 C CNN
 	1    4750 3800
 	1    0    0    -1
@@
 24V_IN
 $Comp
-L DCDC_TDK:i7A24045A033V U2901
+L DCDC_TDK:i7A24045A033V U2
 U 1 1 60E5B9E9
 P 5600 3800
-F 0 "U2901" H 5600 4365 50  0000 C CNN
+F 0 "U2" H 5600 4365 50  0000 C CNN
 F 1 "i7A24045A033V-001-R" H 5600 4274 50  0000 C CNN
-F 2 "" H 5450 4100 50  0001 C CNN
-F 3 "https://product.tdk.com/system/files/dam/doc/product/power/switching-power/dc-dc-converter/catalog/i7a_e.pdf" H 5450 4100 50  0001 C CNN
+F 2 "DCDC:i7A24045A033V" H 5450 4100 50  0001 C CNN
+F 3 "https://product.tdk.com/en/system/files?file=dam/doc/product/power/switching-power/dc-dc-converter/specification/i7a_spec.pdf" H 5450 4100 50  0001 C CNN
 	1    5600 3800
 	1    0    0    -1
@@
 Connection ~ 5000 3950
 Wire Wire Line
-	6800 3650 6800 3500
-Wire Wire Line
-	7450 4000 7450 4100
+	6950 3650 6950 3500
+Wire Wire Line
+	7600 4000 7600 4100
 $Comp
 L power:GND #PWR?
 U 1 1 610D36B1
-P 7450 4200
+P 7600 4200
 AR Path="/5E546572/610D36B1" Ref="#PWR?"  Part="1"
-AR Path="/5E545B2D/610D36B1" Ref="#PWR02902"  Part="1"
+AR Path="/5E545B2D/610D36B1" Ref="#PWR037"  Part="1"
 AR Path="/5E5461C2/610D36B1" Ref="#PWR?"  Part="1"
-F 0 "#PWR02902" H 7450 3950 50  0001 C CNN
-F 1 "GND" H 7455 4027 50  0000 C CNN
-F 2 "" H 7450 4200 50  0001 C CNN
-F 3 "" H 7450 4200 50  0001 C CNN
-	1    7450 4200
+F 0 "#PWR037" H 7600 3950 50  0001 C CNN
+F 1 "GND" H 7605 4027 50  0000 C CNN
+F 2 "" H 7600 4200 50  0001 C CNN
+F 3 "" H 7600 4200 50  0001 C CNN
+	1    7600 4200
 	1    0    0    -1
 $EndComp
@@
 L Device:LED D?
 U 1 1 5E7B7CF5
-P 7450 3850
+P 7600 3850
 AR Path="/5E546572/5E7B7CF5" Ref="D?"  Part="1"
-AR Path="/5E545B2D/5E7B7CF5" Ref="D2901"  Part="1"
+AR Path="/5E545B2D/5E7B7CF5" Ref="D29"  Part="1"
 AR Path="/5E5461C2/5E7B7CF5" Ref="D?"  Part="1"
-F 0 "D2901" V 7550 3700 50  0000 C CNN
-F 1 "PWR_ON_LED" V 7450 3550 50  0000 C CNN
-F 2 "" H 7450 3850 50  0001 C CNN
-F 3 "~" H 7450 3850 50  0001 C CNN
-	1    7450 3850
+F 0 "D29" V 7700 3700 50  0000 C CNN
+F 1 "PWR_ON_LED" V 7600 3550 50  0000 C CNN
+F 2 "" H 7600 3850 50  0001 C CNN
+F 3 "~" H 7600 3850 50  0001 C CNN
+	1    7600 3850
 	0    -1   -1   0
 $EndComp
-Text HLabel 7450 3500 2    70   Output ~ 14
+Text HLabel 7600 3500 2    70   Output ~ 14
 12V_OUT
 Wire Wire Line
-	6500 3650 6500 3500
-Wire Wire Line
-	6800 3950 6800 4100
+	6650 3650 6650 3500
+Wire Wire Line
+	6950 3950 6950 4100
 Connection ~ 4750 3500
 Wire Wire Line
@@
 	4200 3500 4400 3500
 Wire Wire Line
-	6500 4100 6500 3950
+	6650 4100 6650 3950
 $Comp
 L Device:CP C?
 U 1 1 610E5B6D
-P 6800 3800
+P 6950 3800
 AR Path="/5E546572/610E5B6D" Ref="C?"  Part="1"
-AR Path="/5E545B2D/610E5B6D" Ref="C2904"  Part="1"
+AR Path="/5E545B2D/610E5B6D" Ref="C6"  Part="1"
 AR Path="/5E5461C2/610E5B6D" Ref="C?"  Part="1"
-F 0 "C2904" H 6800 4000 50  0000 L CNN
-F 1 "330uF" H 6800 3900 50  0000 L CNN
-F 2 "" H 6838 3650 50  0001 C CNN
-F 3 "~" H 6800 3800 50  0001 C CNN
-	1    6800 3800
+F 0 "C6" H 6950 4000 50  0000 L CNN
+F 1 "330uF" H 6950 3900 50  0000 L CNN
+F 2 "Capacitor_THT:CP_Radial_D10.0mm_P5.00mm" H 6988 3650 50  0001 C CNN
+F 3 "https://content.kemet.com/datasheets/KEM_A4067_A750.pdf" H 6950 3800 50  0001 C CNN
+	1    6950 3800
 	1    0    0    -1
 $EndComp
@@
 L Device:C C?
 U 1 1 5E7CBE12
-P 6500 3800
+P 6650 3800
 AR Path="/5E546572/5E7CBE12" Ref="C?"  Part="1"
-AR Path="/5E545B2D/5E7CBE12" Ref="C2903"  Part="1"
+AR Path="/5E545B2D/5E7CBE12" Ref="C5"  Part="1"
 AR Path="/5E5461C2/5E7CBE12" Ref="C?"  Part="1"
-F 0 "C2903" H 6500 4000 50  0000 L CNN
-F 1 "22µF" H 6500 3900 50  0000 L CNN
-F 2 "" H 6538 3650 50  0001 C CNN
-F 3 "~" H 6500 3800 50  0001 C CNN
-	1    6500 3800
-	1    0    0    -1
-$EndComp
-Wire Wire Line
-	6200 3800 6100 3800
-$Comp
-L Device2:R_Trim R2901
+F 0 "C5" H 6650 4000 50  0000 L CNN
+F 1 "22µF" H 6650 3900 50  0000 L CNN
+F 2 "Capacitor_extra:C_Murata_KCM55" H 6688 3650 50  0001 C CNN
+F 3 "https://search.murata.co.jp/Ceramy/image/img/A01X/G101/ENG/KCM55_E.pdf" H 6650 3800 50  0001 C CNN
+	1    6650 3800
+	1    0    0    -1
+$EndComp
+$Comp
+L Device2:R_Potentiometer_Trim RV1
 U 1 1 60DDD93E
-P 6200 3950
-F 0 "R2901" H 6250 3975 50  0000 L TNN
-F 1 "20kΩ" H 6250 3900 50  0000 L TNN
-F 2 "" V 6130 3950 50  0001 C CNN
-F 3 "~" H 6200 3950 50  0001 C CNN
-	1    6200 3950
-	1    0    0    -1
+P 6300 3800
+F 0 "RV1" H 6250 3800 50  0000 R TNN
+F 1 "50k" H 6250 3900 50  0000 R TNN
+F 2 "" V 6230 3800 50  0001 C CNN
+F 3 "~" H 6300 3800 50  0001 C CNN
+	1    6300 3800
+	-1   0    0    1
 $EndComp
 $Comp
@@
 P 4200 4200
 AR Path="/5E546572/5E7AC91D" Ref="#PWR?"  Part="1"
-AR Path="/5E545B2D/5E7AC91D" Ref="#PWR02901"  Part="1"
+AR Path="/5E545B2D/5E7AC91D" Ref="#PWR036"  Part="1"
 AR Path="/5E5461C2/5E7AC91D" Ref="#PWR?"  Part="1"
-F 0 "#PWR02901" H 4200 3950 50  0001 C CNN
+F 0 "#PWR036" H 4200 3950 50  0001 C CNN
 F 1 "GND" H 4205 4027 50  0000 C CNN
 F 2 "" H 4200 4200 50  0001 C CNN
@@
 Wire Wire Line
 	4200 4100 4200 4200
-Connection ~ 6500 3500
-Connection ~ 6500 4100
-Connection ~ 6800 3500
-Wire Wire Line
-	6800 4100 6500 4100
-Wire Wire Line
-	6500 3500 6800 3500
-Wire Wire Line
-	7450 3650 7450 3700
-Wire Wire Line
-	6800 4100 7450 4100
-Connection ~ 6800 4100
-Connection ~ 7450 4100
-Wire Wire Line
-	7450 3650 7400 3650
+Connection ~ 6650 3500
+Connection ~ 6650 4100
+Connection ~ 6950 3500
+Wire Wire Line
+	6950 4100 6650 4100
+Wire Wire Line
+	6650 3500 6950 3500
+Wire Wire Line
+	7600 3650 7600 3700
+Wire Wire Line
+	6950 4100 7600 4100
+Connection ~ 6950 4100
+Connection ~ 7600 4100
+Wire Wire Line
+	7600 3650 7550 3650
 $Comp
 L Device:R R?
 U 1 1 60E34B0B
-P 7250 3650
+P 7400 3650
 AR Path="/5E546572/60E34B0B" Ref="R?"  Part="1"
-AR Path="/5E545B2D/60E34B0B" Ref="R2903"  Part="1"
+AR Path="/5E545B2D/60E34B0B" Ref="R27"  Part="1"
 AR Path="/5E5461C2/60E34B0B" Ref="R?"  Part="1"
-F 0 "R2903" V 7325 3650 50  0000 C CNN
-F 1 "1.8kΩ" V 7150 3650 50  0000 C CNN
-F 2 "" V 7180 3650 50  0001 C CNN
-F 3 "~" H 7250 3650 50  0001 C CNN
-	1    7250 3650
+F 0 "R27" V 7475 3650 50  0000 C CNN
+F 1 "10k" V 7300 3650 50  0000 C CNN
+F 2 "" V 7330 3650 50  0001 C CNN
+F 3 "~" H 7400 3650 50  0001 C CNN
+	1    7400 3650
 	0    -1   -1   0
 $EndComp
 Wire Wire Line
-	6800 3500 7050 3500
-Wire Wire Line
-	7100 3650 7050 3650
-Wire Wire Line
-	7050 3650 7050 3500
-Connection ~ 7050 3500
-Wire Wire Line
-	7050 3500 7450 3500
-Wire Wire Line
-	6100 4100 6200 4100
-Wire Wire Line
-	7450 4100 7450 4200
-Connection ~ 6200 4100
-Wire Wire Line
-	6200 4100 6500 4100
+	6950 3500 7200 3500
+Wire Wire Line
+	7250 3650 7200 3650
+Wire Wire Line
+	7200 3650 7200 3500
+Connection ~ 7200 3500
+Wire Wire Line
+	7200 3500 7600 3500
+Wire Wire Line
+	7600 4100 7600 4200
 Connection ~ 6350 3500
 Wire Wire Line
-	6350 3500 6500 3500
+	6350 3500 6650 3500
 Wire Wire Line
 	6200 3500 6350 3500
+Wire Wire Line
+	6100 4100 6300 4100
+Wire Wire Line
+	6300 3950 6300 4100
+Connection ~ 6300 4100
+Wire Wire Line
+	6300 4100 6650 4100
+Wire Wire Line
+	6150 3800 6100 3800
+NoConn ~ 6300 3650
 $EndSCHEMATC

Commit message: rPDM - Started on board layout
Parts:
- D3: renamed from D29; footprint (none) -> Diode_SMD:D_0603_1608Metric_Pad1.05x0.95mm_HandSolder
- R1: renamed from R27; footprint (none) -> Resistor_SMD:R_0805_2012Metric_Pad1.15x1.40mm_HandSolder
- renumbered C3 to C1, C4 to C2, C5 to C3, C6 to C4, U2 to U1
Changed lines of the file:
@@
 $Descr A4 11693 8268
 encoding utf-8
-Sheet 30 32
+Sheet 3 32
 Title "DC/DC Converter Circuit"
 Date "2021-06-28"
@@
 P 4400 3800
 AR Path="/5E546572/5E7A7C2F" Ref="C?"  Part="1"
-AR Path="/5E545B2D/5E7A7C2F" Ref="C3"  Part="1"
+AR Path="/5E545B2D/5E7A7C2F" Ref="C1"  Part="1"
 AR Path="/5E5461C2/5E7A7C2F" Ref="C?"  Part="1"
-F 0 "C3" H 4400 4000 50  0000 L CNN
+F 0 "C1" H 4400 4000 50  0000 L CNN
 F 1 "330µF" H 4400 3900 50  0000 L CNN
 F 2 "Capacitor_THT:CP_Radial_D10.0mm_P5.00mm" H 4438 3650 50  0001 C CNN
@@
 P 4750 3800
 AR Path="/5E546572/5E7A88E4" Ref="C?"  Part="1"
-AR Path="/5E545B2D/5E7A88E4" Ref="C4"  Part="1"
+AR Path="/5E545B2D/5E7A88E4" Ref="C2"  Part="1"
 AR Path="/5E5461C2/5E7A88E4" Ref="C?"  Part="1"
-F 0 "C4" H 4750 4000 50  0000 L CNN
+F 0 "C2" H 4750 4000 50  0000 L CNN
 F 1 "22µF" H 4750 3900 50  0000 L CNN
 F 2 "Capacitor_extra:C_Murata_KCM55" H 4788 3650 50  0001 C CNN
@@
 24V_IN
 $Comp
-L DCDC_TDK:i7A24045A033V U2
+L DCDC_TDK:i7A24045A033V U1
 U 1 1 60E5B9E9
 P 5600 3800
-F 0 "U2" H 5600 4365 50  0000 C CNN
+F 0 "U1" H 5600 4365 50  0000 C CNN
 F 1 "i7A24045A033V-001-R" H 5600 4274 50  0000 C CNN
 F 2 "DCDC:i7A24045A033V" H 5450 4100 50  0001 C CNN
@@
 P 7600 4200
 AR Path="/5E546572/610D36B1" Ref="#PWR?"  Part="1"
-AR Path="/5E545B2D/610D36B1" Ref="#PWR037"  Part="1"
+AR Path="/5E545B2D/610D36B1" Ref="#PWR06"  Part="1"
 AR Path="/5E5461C2/610D36B1" Ref="#PWR?"  Part="1"
-F 0 "#PWR037" H 7600 3950 50  0001 C CNN
+F 0 "#PWR06" H 7600 3950 50  0001 C CNN
 F 1 "GND" H 7605 4027 50  0000 C CNN
 F 2 "" H 7600 4200 50  0001 C CNN
@@
 P 7600 3850
 AR Path="/5E546572/5E7B7CF5" Ref="D?"  Part="1"
-AR Path="/5E545B2D/5E7B7CF5" Ref="D29"  Part="1"
+AR Path="/5E545B2D/5E7B7CF5" Ref="D3"  Part="1"
 AR Path="/5E5461C2/5E7B7CF5" Ref="D?"  Part="1"
-F 0 "D29" V 7700 3700 50  0000 C CNN
+F 0 "D3" V 7700 3700 50  0000 C CNN
 F 1 "PWR_ON_LED" V 7600 3550 50  0000 C CNN
-F 2 "" H 7600 3850 50  0001 C CNN
+F 2 "Diode_SMD:D_0603_1608Metric_Pad1.05x0.95mm_HandSolder" H 7600 3850 50  0001 C CNN
 F 3 "~" H 7600 3850 50  0001 C CNN
 	1    7600 3850
@@
 P 6950 3800
 AR Path="/5E546572/610E5B6D" Ref="C?"  Part="1"
-AR Path="/5E545B2D/610E5B6D" Ref="C6"  Part="1"
+AR Path="/5E545B2D/610E5B6D" Ref="C4"  Part="1"
 AR Path="/5E5461C2/610E5B6D" Ref="C?"  Part="1"
-F 0 "C6" H 6950 4000 50  0000 L CNN
+F 0 "C4" H 6950 4000 50  0000 L CNN
 F 1 "330uF" H 6950 3900 50  0000 L CNN
 F 2 "Capacitor_THT:CP_Radial_D10.0mm_P5.00mm" H 6988 3650 50  0001 C CNN
@@
 P 6650 3800
 AR Path="/5E546572/5E7CBE12" Ref="C?"  Part="1"
-AR Path="/5E545B2D/5E7CBE12" Ref="C5"  Part="1"
+AR Path="/5E545B2D/5E7CBE12" Ref="C3"  Part="1"
 AR Path="/5E5461C2/5E7CBE12" Ref="C?"  Part="1"
-F 0 "C5" H 6650 4000 50  0000 L CNN
+F 0 "C3" H 6650 4000 50  0000 L CNN
 F 1 "22µF" H 6650 3900 50  0000 L CNN
 F 2 "Capacitor_extra:C_Murata_KCM55" H 6688 3650 50  0001 C CNN
@@
 P 4200 4200
 AR Path="/5E546572/5E7AC91D" Ref="#PWR?"  Part="1"
-AR Path="/5E545B2D/5E7AC91D" Ref="#PWR036"  Part="1"
+AR Path="/5E545B2D/5E7AC91D" Ref="#PWR05"  Part="1"
 AR Path="/5E5461C2/5E7AC91D" Ref="#PWR?"  Part="1"
-F 0 "#PWR036" H 4200 3950 50  0001 C CNN
+F 0 "#PWR05" H 4200 3950 50  0001 C CNN
 F 1 "GND" H 4205 4027 50  0000 C CNN
 F 2 "" H 4200 4200 50  0001 C CNN
@@
 P 7400 3650
 AR Path="/5E546572/60E34B0B" Ref="R?"  Part="1"
-AR Path="/5E545B2D/60E34B0B" Ref="R27"  Part="1"
+AR Path="/5E545B2D/60E34B0B" Ref="R1"  Part="1"
 AR Path="/5E5461C2/60E34B0B" Ref="R?"  Part="1"
-F 0 "R27" V 7475 3650 50  0000 C CNN
+F 0 "R1" V 7475 3650 50  0000 C CNN
 F 1 "10k" V 7300 3650 50  0000 C CNN
-F 2 "" V 7330 3650 50  0001 C CNN
+F 2 "Resistor_SMD:R_0805_2012Metric_Pad1.15x1.40mm_HandSolder" V 7330 3650 50  0001 C CNN
 F 3 "~" H 7400 3650 50  0001 C CNN
 	1    7400 3650
