File: LV/RPDM v2/RPDM v2.sch (KiCad schematic (older format))
At the start: 4 parts

Commit message: RPDM v2 nearly done
Parts:
- removed J?: Conn_02x04_Counter_Clockwise, symbol Connector_Generic:Conn_02x04_Counter_Clockwise
- added J?: CONN_LV_BATT, symbol Connector_Generic:Conn_02x01
- TP?: value TestPoint -> GND Test Point
Connections:
- net labels added: 5V, ACCUMULATOR, ACC_FAN_1, ACC_FAN_2, ACC_FAN_3, BMS_DATALOGGER, BRAKE_LIGHT, HV_DIST, INTERLOCK, LV_BATT_NEG, LV_BATT_POS, MOTOR_CONTROLLER_1, MOTOR_CONTROLLER_2, PDOC, PUMP_1, PUMP_1_Trigger, PUMP_2, RAD_FAN_1, RAD_FAN_1_Trigger, RAD_FAN_2, SPARE_RELAY_1, SPARE_RELAY_2, SPARE_Trigger_1, SPARE_Trigger_2, TSAL
- net labels removed: 5V_Out1, 5V_Out2, Fuse_1, Fuse_10, Fuse_11, Fuse_12, Fuse_13, Fuse_2, Fuse_3, Fuse_4, Fuse_5, Fuse_6, Fuse_7, Fuse_8, Fuse_9, Relay_1, Relay_2, Relay_3, Relay_4, Relay_Trigger_1, Relay_Trigger_2, Relay_Trigger_3, Relay_Trigger_4
- wire segments 106 -> 156
- no-connect marks 2 -> 0
Other:
- note removed: "From Battery"
- note removed: "GND Test Point"
- moved on the sheet: J?, TP?

Commit message: RPDM update
Parts:
- added TP?: GND Test Point, symbol Connector:TestPoint
Connections:
- net labels added: 5V_GND, ACCUMULATOR_GND, ACC_FAN_1_GND, ACC_FAN_2_GND, ACC_FAN_3_GND, BATT_I, BATT_V, BMS_DATALOGGER_GND, FPDM_GND, HV_DIST_GND, INTERLOCK_BUTTONS_GND, INTERLOCK_GND, MOTOR_CONTROLLER_1_GND, MOTOR_CONTROLLER_2_GND, PDOC_12V, PUMP_1_GND, PUMP_2_GND, RAD_FAN_1_GND, RAD_FAN_2_GND, RAD_FAN_Trigger, SPARE_RELAY_1_GND, SPARE_RELAY_2_GND, TSAL_GND
- net labels removed: DCDC_I, DCDC_V, Fuse_14, PDOC, RAD_FAN_1_Trigger
- wire segments 156 -> 91
Other:
- moved on the sheet: J?, TP?

Commit message: rpdm
Parts:
- removed J?: CONN_LV_BATT, symbol Connector_Generic:Conn_02x01
- added C? (x2): 10uF, symbol Device:C
- added C?: 10nF, symbol Device:C
- added J101: 24V_IN, symbol Connector_Generic:Conn_01x03
- added Q?: Q_NPN_BCE, symbol Device:Q_NPN_BCE
- added R?: 470, symbol Device:R
- added R? (x5): 10k, symbol Device:R
- added R?: 1.8k, symbol Device:R
- added RV?: 20kΩ, symbol Device2:R_Potentiometer_Trim
- added TP102: GND Test Point, symbol Connector:TestPoint
- added U?: LM555, symbol Timer:LM555
- gave numbers to parts that had none: 4
Connections:
- net labels added: +12V, +24V_BATT, +24V_EXT, -24V, 555_Out, 555_Trigger, Green_Out, Red_Out, Vin
- net labels removed: LV_BATT_NEG, LV_BATT_POS
- wire segments 91 -> 140
Other:
- note added: "Frequency Adjust, appox. 2.3-6.6Hz"
- note added: "Power Distribution"
- note added: "TSAL Flash Circuit"
- note added: "TSAL Logic Outputs"
- note added: "TSAT Trigger Logic"
- moved on the sheet: J102, J103, TP101, TP103

Commit message: rpdm
Parts:
- removed C? (x2): 10uF, symbol Device:C
- removed C?: 10nF, symbol Device:C
- removed J103: 776180-1, TE_776180-1, symbol 776180-1:776180-1
- removed Q?: Q_NPN_BCE, symbol Device:Q_NPN_BCE
- removed R?: 470, symbol Device:R
- removed R? (x5): 10k, symbol Device:R
- removed R?: 1.8k, symbol Device:R
- removed RV?: 20kΩ, symbol Device2:R_Potentiometer_Trim
- removed U?: LM555, symbol Timer:LM555
- added J?: 1-770669-1, TE_1-770669-1, symbol 1-770669-1:1-770669-1
Connections:
- net labels added: 12V, RELAY_1, RELAY_2, RELAY_3, RELAY_4
- net labels removed: +12V, 555_Out, 555_Trigger, Green_Out, Red_Out, Vin
- wire segments 140 -> 162
Other:
- note added: "Convert to 12V"
- note added: "GLV power in (18-25V)"
- note added: "Measure Current/Voltage"
- note added: "Power Entry"
- note removed: "Frequency Adjust, appox. 2.3-6.6Hz"
- note removed: "Power Distribution"
- note removed: "TSAL Flash Circuit"
- note removed: "TSAL Logic Outputs"
- note removed: "TSAT Trigger Logic"
- moved on the sheet: J101, J102, TP101, TP102, TP103

Commit message: rpdm
Parts:
- J2: renamed from J?; footprint TE_1-770669-1 -> 1-770669-1:TE_1-770669-1
- J3: renamed from J102; footprint TE_776180-1 -> 776180-1:TE_776180-1
- TP1: renamed from TP101; footprint (none) -> TestPoint:TestPoint_THTPad_1.0x1.0mm_Drill0.5mm
- TP2: renamed from TP102; value GND Test Point -> Ext. power test point; footprint (none) -> TestPoint:TestPoint_THTPad_1.0x1.0mm_Drill0.5mm
- TP3: renamed from TP103; value GND Test Point -> Battery test point; footprint (none) -> TestPoint:TestPoint_THTPad_1.0x1.0mm_Drill0.5mm
- renumbered J101 to J1
Connections:
- net TSAT_Trigger is gone; now on net BATT_I: J2.10
- net 5V: now also J3.16; no longer J2.1
- net BATT_I: no longer J2.12
- net BATT_V: now also J2.9; no longer J2.11
- net BRAKE_LIGHT: now also J3.17; no longer J2.2
- net GND: now also J2.6, J2.7, J2.8; no longer J2.13, J2.15, J2.17, J2.18, J2.19, J3.18
- net PDOC_12V: now also J3.18; no longer J2.3
- net PUMP_1_Trigger: now also J2.2; no longer J2.5
- net RAD_FAN_Trigger: now also J2.1; no longer J2.4
- net SPARE_RELAY_1: now also J2.13; no longer J3.16
- net SPARE_RELAY_2: now also J2.15; no longer J3.17
- net SPARE_Trigger_1: now also J2.3; no longer J2.6
- net SPARE_Trigger_2: now also J2.4; no longer J2.7
- net TSAL_Green: now also J2.12; no longer J2.9
- net TSAL_Red: now also J2.11; no longer J2.8
- net PUMP_1 renamed PUMPS
- net RAD_FAN_1 renamed RAD_FANS
- new net SPARE_FUSE_1: J2.17
- new net SPARE_FUSE_2: J2.18
- new net SPARE_FUSE_3: J2.19
- new net TSAT: J2.5
Other:
- moved on the sheet: J2, J3

Commit message: rPDM - Started on board layout
Connections:
- net labels added: 5V_DCDC
- wire segments 132 -> 130
Other:
- moved on the sheet: J1, J2, J3

Commit message: RPDM
Parts:
- J1: footprint (none) -> UOWM_TerminalBlocks:EB167A-03-M; symbol Connector_Generic:Conn_01x03 -> Connector:Screw_Terminal_01x03
- J2: footprint 1-770669-1:TE_1-770669-1 -> UOWM_Connectors:TE_1-770669-1
- J3: footprint 776180-1:TE_776180-1 -> UOWM_Connectors:TE_1-770669-1; symbol 776180-1:776180-1 -> 1-770669-1:1-770669-1
Connections:
- net labels added: 24_DCDC_IN, 24_ISENSE_IN, ACC_FANS, TSAL_PWR
- net labels removed: ACC_FAN_3, ACC_FAN_3_GND, PUMP_1, PUMP_2, PUMP_2_GND, RAD_FAN_1, RAD_FAN_2, RAD_FAN_2_GND, SPARE_FUSE_3, SPARE_FUSE_3_GND, TSAL
- wire segments 130 -> 115
Other:
- note added: "10A->"
- note added: "20A->"
- note added: "2A->"
- note added: "4A->"
- note added: "External power switching"
- moved on the sheet: J2, TP1, TP2, TP3

Commit message: RPDM nearly finished
Connections:
- net +24V_BATT: now also J1.2 (Pin_2), TP2.1; no longer J1.1 (Pin_1), TP3.1
- net +24V_EXT: now also J1.3 (Pin_3), TP3.1; no longer J1.2 (Pin_2), TP2.1
- net GND: now also J1.1 (Pin_1); no longer J1.3 (Pin_3)
Other:
- moved on the sheet: J1, TP1, TP2, TP3
