File: LV/RPDM v2/Fuse.sch (KiCad schematic (older format))
At the start: 3 parts

Commit message: RPDM nearly finished
Changed lines of the file:
@@
 $Descr A4 11693 8268
 encoding utf-8
-Sheet 4 30
+Sheet 11 30
 Title "Fuse Circuit"
 Date "2021-06-28"
@@
 AR Path="/5E553C05/618E952A/5E574E2C" Ref="F19"  Part="1"
 AR Path="/5E553C05/618E952E/5E574E2C" Ref="F20"  Part="1"
-F 0 "F1" V 5750 3050 50  0000 L CNN
+F 0 "F8" V 5750 3050 50  0000 L CNN
 F 1 "Fuse" V 5950 3100 50  0000 L CNN
 F 2 "UOWM_Fuses:Keystone_3568" V 5780 3150 50  0001 C CNN
@@
 AR Path="/5E553C05/618E952A/5E57CF75" Ref="#PWR040"  Part="1"
 AR Path="/5E553C05/618E952E/5E57CF75" Ref="#PWR041"  Part="1"
-F 0 "#PWR022" H 6250 3800 50  0001 C CNN
+F 0 "#PWR029" H 6250 3800 50  0001 C CNN
 F 1 "GND" H 6255 3877 50  0000 C CNN
 F 2 "" H 6250 4050 50  0001 C CNN
@@
 AR Path="/5E553C05/618E952A/5E5770E7" Ref="R34"  Part="1"
 AR Path="/5E553C05/618E952E/5E5770E7" Ref="R35"  Part="1"
-F 0 "R16" H 6450 3350 50  0000 C CNN
+F 0 "R23" H 6450 3350 50  0000 C CNN
 F 1 "10k" H 6400 3450 50  0000 C CNN
 F 2 "Resistor_SMD:R_0805_2012Metric_Pad1.15x1.40mm_HandSolder" V 6180 3400 50  0001 C CNN
@@
 AR Path="/5E553C05/618E952A/5E57B77F" Ref="D27"  Part="1"
 AR Path="/5E553C05/618E952E/5E57B77F" Ref="D28"  Part="1"
-F 0 "D9" V 6300 4050 50  0000 C CNN
+F 0 "D16" V 6300 4050 50  0000 C CNN
 F 1 "OK_LED" V 6200 4050 50  0000 C CNN
 F 2 "Diode_SMD:D_0603_1608Metric_Pad1.05x0.95mm_HandSolder" H 6250 3800 50  0001 C CNN

Commit message: RPDM
Changed lines of the file:
@@
 $Descr A4 11693 8268
 encoding utf-8
-Sheet 11 30
+Sheet 8 30
 Title "Fuse Circuit"
 Date "2021-06-28"
@@
 AR Path="/5E553C05/618E952A/5E574E2C" Ref="F19"  Part="1"
 AR Path="/5E553C05/618E952E/5E574E2C" Ref="F20"  Part="1"
-F 0 "F8" V 5750 3050 50  0000 L CNN
+F 0 "F5" V 5750 3050 50  0000 L CNN
 F 1 "Fuse" V 5950 3100 50  0000 L CNN
 F 2 "UOWM_Fuses:Keystone_3568" V 5780 3150 50  0001 C CNN
@@
 AR Path="/5E553C05/618E952A/5E57CF75" Ref="#PWR040"  Part="1"
 AR Path="/5E553C05/618E952E/5E57CF75" Ref="#PWR041"  Part="1"
-F 0 "#PWR029" H 6250 3800 50  0001 C CNN
+F 0 "#PWR026" H 6250 3800 50  0001 C CNN
 F 1 "GND" H 6255 3877 50  0000 C CNN
 F 2 "" H 6250 4050 50  0001 C CNN
@@
 AR Path="/5E553C05/618E952A/5E5770E7" Ref="R34"  Part="1"
 AR Path="/5E553C05/618E952E/5E5770E7" Ref="R35"  Part="1"
-F 0 "R23" H 6450 3350 50  0000 C CNN
+F 0 "R20" H 6450 3350 50  0000 C CNN
 F 1 "10k" H 6400 3450 50  0000 C CNN
 F 2 "Resistor_SMD:R_0805_2012Metric_Pad1.15x1.40mm_HandSolder" V 6180 3400 50  0001 C CNN
@@
 AR Path="/5E553C05/618E952A/5E57B77F" Ref="D27"  Part="1"
 AR Path="/5E553C05/618E952E/5E57B77F" Ref="D28"  Part="1"
-F 0 "D16" V 6300 4050 50  0000 C CNN
+F 0 "D13" V 6300 4050 50  0000 C CNN
 F 1 "OK_LED" V 6200 4050 50  0000 C CNN
 F 2 "Diode_SMD:D_0603_1608Metric_Pad1.05x0.95mm_HandSolder" H 6250 3800 50  0001 C CNN
