File: LV/LV Harness/LV_Harness/LV_Harness.sch (KiCad schematic (older format))
At the start: 0 parts

Commit message: started LV Harness
Parts:
- added J?: Plug A, symbol Connector:Conn_01x12_Female
- added J?: Plug B, symbol Connector:Conn_01x12_Female
- added J? (x2): Conn_01x12_Male, symbol Connector:Conn_01x12_Male
- added J? (x4): Conn_01x03_Female, symbol Connector:Conn_01x03_Female
- added J? (x4): Conn_01x03_Male, symbol Connector:Conn_01x03_Male
- added J?: Conn_01x35_Male, symbol Connector:Conn_01x35_Male
- added J?: Conn_01x35_Female, symbol Connector:Conn_01x35_Female
Connections:
- net labels added: 12V, 3.3V, 5V, AMP_OUT, BMS_CHG, BMS_GND, BMS_OK, BMS_RDY, CAN1+, CAN1-, CAN2+, CAN2-, CHG_OK, DASH-3, DCH_OK, ECU-A4, ECU-A5, ECU-A6, ECU-A7, ECU-A8, ECU-A9, FAN_EN, FAN_MON, FAN_PWM, FL_WSS, FPDM-1, FPDM-3, FR_WSS, F_BPS, GND, IMD_OK, IMD_PWM, INTERLOCK, MP1_IN, MP1_OUT, PDOC_IN, PDOC_OUT, RPDM-1, RTD_IN, RTD_LED, R_BPS, SAS, Sense, TEST_IN, TEST_OUT, THERM_4, TPS_1, TPS_2, TPS_3.3V, TPS_GND, Un-populated, V_CHECK
- wire segments 0 -> 175
Other:
- note added: "Ampseal 35 PLU"
- note added: "Ampseal 35 REC"
- note added: "BMS Main I/O"
- note added: "DTM 3P REC"
- note added: "DTM 3S PLG"
- note added: "ECU"
- note added: "F_BPS"
- note added: "IMD"
- note added: "LV Harness"
- note added: "Plug A"
- note added: "Plug B"
- note added: "Pre-Charge"
- note added: "R_BPS"
- note added: "TEST_LOOP"
- note added: "TPS_1"
- note added: "TPS_2"

Commit message: harness
Parts:
- added J? (x2): Conn_01x23_Male, symbol Connector:Conn_01x23_Male
- added J? (x2): Conn_01x23_Female, symbol Connector:Conn_01x23_Female
Connections:
- net labels added: 5V_GND, ACCUMULATOR, ACCUMULATOR_GND, ACC_FANS, ACC_FAN_1, ACC_FAN_1_GND, ACC_FAN_2, ACC_FAN_2_GND, BATT_I, BATT_V, BMS_DATALOGGER, BMS_DATALOGGER_GND, BRAKE_LIGHT, FPDM, FPDM_GND, HV_DIST, HV_DIST_GND, INTERLOCK_BUTTONS_GND, INTERLOCK_GND, MOTOR_CONTROLLER_1, MOTOR_CONTROLLER_1_GND, MOTOR_CONTROLLER_2, MOTOR_CONTROLLER_2_GND, PDOC_12V, PUMPS, PUMP_1_GND, PUMP_1_Trigger, RAD_FANS, RAD_FAN_1_GND, RAD_FAN_Trigger, SPARE_FUSE_1, SPARE_FUSE_1_GND, SPARE_FUSE_2, SPARE_FUSE_2_GND, SPARE_RELAY_1, SPARE_RELAY_1_GND, SPARE_RELAY_2, SPARE_RELAY_2_GND, SPARE_Trigger_1, SPARE_Trigger_2, TSAL_GND, TSAL_Green, TSAL_PWR, TSAL_Red, TSAT
- net labels removed: Un-populated
- wire segments 175 -> 224
- no-connect marks 0 -> 17

Commit message: harness
Parts:
- removed J?: Plug A, symbol Connector:Conn_01x12_Female
- removed J?: Plug B, symbol Connector:Conn_01x12_Female
- removed J? (x2): Conn_01x12_Male, symbol Connector:Conn_01x12_Male
- added J?: Conn_01x14_Female, symbol Connector:Conn_01x14_Female
- added J?: Conn_01x14_Male, symbol Connector:Conn_01x14_Male
- added J?: Conn_01x09_Female, symbol Connector:Conn_01x08_Female
- added J?: Conn_01x09_Male, symbol Connector:Conn_01x08_Male
- added J?: Conn_01x35_Female, symbol Connector:Conn_01x35_Female
- added J?: Conn_01x35_Male, symbol Connector:Conn_01x35_Male
Connections:
- net labels added: FPDM-xx, PWM, RPDM-A07, RPDM-B08, fan1_12V, fan1_GND, fan2_12V, fan2_GND, fan3_12V, fan3_GND, monitor
- wire segments 224 -> 261
Other:
- note removed: "Plug A"
- note removed: "Plug B"
- moved on the sheet: J?
