File: LV/LV Harness/LV_Harness/Connector_Sheets/Acc_Fan_Pinout/Acc_Fan_Pinout.sch (KiCad schematic (older format))
At the start: 6 parts

Commit message: Changes to LV Harness Folders
Parts:
- removed J? (x3): Conn_01x03_Female, symbol Connector:Conn_01x03_Female
- removed J? (x3): Conn_01x03_Male, symbol Connector:Conn_01x03_Male
Changed lines of the file:
@@
 EESchema Schematic File Version 4
+LIBS:Acc_Fan_Pinout-cache
 EELAYER 29 0
 EELAYER END
@@
 Comment4 ""
 $EndDescr
-$Comp
-L Connector:Conn_01x03_Female J?
-U 1 1 60F25F94
-P 5750 3250
-F 0 "J?" H 5600 3500 50  0001 L CNN
-F 1 "Conn_01x03_Female" H 5050 3050 50  0001 L CNN
-F 2 "" H 5750 3250 50  0001 C CNN
-F 3 "~" H 5750 3250 50  0001 C CNN
-	1    5750 3250
-	1    0    0    -1
-$EndComp
-$Comp
-L Connector:Conn_01x03_Male J?
-U 1 1 60F2639B
-P 5750 3250
-F 0 "J?" H 5850 3500 50  0001 C CNN
-F 1 "Conn_01x03_Male" H 6050 3050 50  0001 C CNN
-F 2 "" H 5750 3250 50  0001 C CNN
-F 3 "~" H 5750 3250 50  0001 C CNN
-	1    5750 3250
-	1    0    0    -1
-$EndComp
-$Comp
-L Connector:Conn_01x03_Female J?
-U 1 1 60F281BC
-P 5750 3750
-F 0 "J?" H 5600 4000 50  0001 L CNN
-F 1 "Conn_01x03_Female" H 5050 3550 50  0001 L CNN
-F 2 "" H 5750 3750 50  0001 C CNN
-F 3 "~" H 5750 3750 50  0001 C CNN
-	1    5750 3750
-	1    0    0    -1
-$EndComp
-$Comp
-L Connector:Conn_01x03_Male J?
-U 1 1 60F281C2
-P 5750 3750
-F 0 "J?" H 5850 4000 50  0001 C CNN
-F 1 "Conn_01x03_Male" H 6050 3550 50  0001 C CNN
-F 2 "" H 5750 3750 50  0001 C CNN
-F 3 "~" H 5750 3750 50  0001 C CNN
-	1    5750 3750
-	1    0    0    -1
-$EndComp
-$Comp
-L Connector:Conn_01x03_Female J?
-U 1 1 60F2B94C
-P 5750 4250
-F 0 "J?" H 5600 4500 50  0001 L CNN
-F 1 "Conn_01x03_Female" H 5050 4050 50  0001 L CNN
-F 2 "" H 5750 4250 50  0001 C CNN
-F 3 "~" H 5750 4250 50  0001 C CNN
-	1    5750 4250
-	1    0    0    -1
-$EndComp
-$Comp
-L Connector:Conn_01x03_Male J?
-U 1 1 60F2B952
-P 5750 4250
-F 0 "J?" H 5850 4500 50  0001 C CNN
-F 1 "Conn_01x03_Male" H 6050 4050 50  0001 C CNN
-F 2 "" H 5750 4250 50  0001 C CNN
-F 3 "~" H 5750 4250 50  0001 C CNN
-	1    5750 4250
-	1    0    0    -1
-$EndComp
 $EndSCHEMATC
